Commit message: working with robot3.urdf

File: urdf/robot.urdf (robot description, URDF)
Before this commit: robot Self_Balancing_Robot, 3 links, 2 joints
Links:
- link Chassis: geometry collision box size=0.075 0.175 0.157; visual mesh filename=/home/glauberrleite/dev/tcc/self_balancing_robot/urdf/meshe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
- link Left_Wheel: geometry collision cylinder length=0.037 radius=0.0316; visual mesh filename=/home/glauberrleite/dev/tcc/self_balancing_robot/urdf/meshe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
- link Right_Wheel: geometry collision cylinder length=0.037 radius=0.0316; visual mesh filename=/home/glauberrleite/dev/tcc/self_balancing_robot/urdf/meshe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
